File: FlashSD.kicad_sch (KiCad schematic)
At the start: 0 parts

Commit message: finalizing schematic
Parts:
- added D3: SRV05-4.TCT, myFootprints:SOT95P280X145-6N, symbol SRV05-4.TCT:SRV05-4.TCT
- added J4: Micro_SD_Card, Connector_Card:microSD_HC_Molex_104031-0811, symbol Connector:Micro_SD_Card
- added R10: 220R, Resistor_SMD:R_0805_2012Metric_Pad1.20x1.40mm_HandSolder, symbol Device:R
- added R9: 10k, Resistor_SMD:R_0805_2012Metric_Pad1.20x1.40mm_HandSolder, symbol Device:R
Connections:
- new net: J4.2 (DAT3/CD), R9.2
- new net: J4.5 (CLK), R10.2
- new net +3.3V: D3.5, J4.4 (VDD), R9.1
- new net GND: D3.2, J4.6 (VSS), J4.9 (SHIELD)
- new net SDCLK: R10.1
- new net SDMISO: D3.4, J4.3 (CMD)
- new net SDMOSI: D3.6, J4.7 (DAT0)
- no-connect marks 0 -> 4
