File: MCU.kicad_sch (KiCad schematic)
At the start: 28 parts, among them J1 Microsemi_FlashPro-JTAG-10, U1 STM32F405RGT6, Y1 8mhz

Commit message: finalizing schematic
Parts:
- renumbered C1 to C24, C2 to C25, C3 to C26, C4 to C27, C5 to C28, C6 to C29, C7 to C30, C8 to C31, C9 to C32, C10 to C33, C11 to C34, C12 to C35, C13 to C36, C14 to C37, C15 to C38, FB1 to FB2, J1 to J2, R1 to R3, R2 to R4, R3 to R5, R4 to R6, U1 to U2, Y1 to Y2
Connections:
- net SPI_SCK: now reaches U2.21 (PA5)
- net SPI_MISO: now reaches U2.22 (PA6)
- net SPI_MOSI: now reaches U2.23 (PA7)
- net SxDIO1: now reaches U2.39 (PC8)
- net SxNSS: now reaches U2.51 (PC10)
- net SxReset: now reaches U2.52 (PC11)
- net SxBusy: now reaches U2.53 (PC12)
- net DrougeADC: no longer names the net of U2.25 (PC5)
- net GPS1_RX: no longer names the net of U2.30 (PB11)
- net GPS1_TX renamed SPI2_SCK
- net GPS2_RX: no longer names the net of U2.37 (PC6)
- net GPS2_TX: no longer names the net of U2.38 (PC7)
- net I2CSDA: no longer names the net of U2.58 (PB6)
- net I2CSDL: no longer names the net of U2.59 (PB7)
- net PyroADC: no longer names the net of U2.15 (PA1)
- net SPI2-MISO renamed SPI2_MOSI
- net SPI2-MOSI renamed SPI2_MISO
- no-connect marks 39 -> 40
