File: USB_C.kicad_sch (KiCad schematic)
At the start: 4 parts, among them J2 USB_C_Receptacle

Commit message: finalizing schematic
Parts:
- gave numbers to parts that had none: 1
- renumbered J2 to J3, R5 to R7, R6 to R8
Changed lines of the file:
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@@
+		(color 0 0 0 0)
+	)
+	(junction
+		(at 59.69 26.67)
+		(diameter 0)
 		(color 0 0 0 0)
 	)
@@
 	(wire
 		(pts
-			(xy 53.34 26.67) (xy 71.12 26.67)
+			(xy 53.34 26.67) (xy 59.69 26.67)
 		)
 		(stroke
@@
 	(wire
 		(pts
+			(xy 59.69 26.67) (xy 71.12 26.67)
+		)
+		(stroke
+			(width 0)
+			(type default)
+		)
+	)
+	(wire
+		(pts
 			(xy 62.23 40.64) (xy 63.5 40.64)
 		)
@@
 		)
 	)
-	(global_label "D-"
+	(hierarchical_label "D-"
 		(shape input)
 		(at 63.5 40.64 0)
-		(fields_autoplaced yes)
 		(effects
 			(font
@@
 			(justify left)
 		)
-		(property "Intersheetrefs" "${INTERSHEET_REFS}"
-			(at 69.3276 40.64 0)
-			(effects
-				(font
-					(size 1.27 1.27)
-				)
-				(justify left)
-				(hide yes)
-			)
-		)
-	)
-	(global_label "D+"
+	)
+	(hierarchical_label "VBUS"
 		(shape input)
-		(at 66.04 49.53 0)
-		(fields_autoplaced yes)
+		(at 68.58 26.67 90)
 		(effects
 			(font
@@
 			(justify left)
 		)
-		(property "Intersheetrefs" "${INTERSHEET_REFS}"
-			(at 71.8676 49.53 0)
-			(effects
-				(font
-					(size 1.27 1.27)
-				)
-				(justify left)
-				(hide yes)
-			)
+	)
+	(hierarchical_label "D+"
+		(shape input)
+		(at 66.04 49.53 0)
+		(effects
+			(font
+				(size 1.27 1.27)
+			)
+			(justify left)
 		)
 	)
@@
 		(on_board yes)
 		(dnp no)
-		(property "Reference" "#PWR036"
+		(property "Reference" "#PWR057"
 			(at 91.44 40.64 0)
 			(effects
@@
 			(project "sx1262xBoard"
 				(path "/e72bc999-a506-4a63-8c4b-c84561b55f6d/3bb3cd23-0a7e-4579-8d0d-52812beb7407"
-					(reference "#PWR036")
+					(reference "#PWR057")
 					(unit 1)
 				)
@@
 		(dnp no)
 		(fields_autoplaced yes)
-		(property "Reference" "D?"
+		(property "Reference" "D2"
 			(at 82.55 50.8 0)
 			(effects
@@
 			(project "sx1262xBoard"
 				(path "/e72bc999-a506-4a63-8c4b-c84561b55f6d/3bb3cd23-0a7e-4579-8d0d-52812beb7407"
-					(reference "D?")
+					(reference "D2")
 					(unit 1)
 				)
@@
 		(dnp no)
 		(fields_autoplaced yes)
-		(property "Reference" "#PWR038"
+		(property "Reference" "#PWR059"
 			(at 116.84 46.99 0)
 			(effects
@@
 			(project "sx1262xBoard"
 				(path "/e72bc999-a506-4a63-8c4b-c84561b55f6d/3bb3cd23-0a7e-4579-8d0d-52812beb7407"
-					(reference "#PWR038")
+					(reference "#PWR059")
 					(unit 1)
 				)
@@
 		(dnp no)
 		(fields_autoplaced yes)
-		(property "Reference" "#PWR034"
+		(property "Reference" "#PWR055"
 			(at 67.31 26.67 0)
 			(effects
@@
 			(project "sx1262xBoard"
 				(path "/e72bc999-a506-4a63-8c4b-c84561b55f6d/3bb3cd23-0a7e-4579-8d0d-52812beb7407"
-					(reference "#PWR034")
+					(reference "#PWR055")
+					(unit 1)
+				)
+			)
+		)
+	)
+	(symbol
+		(lib_id "power:PWR_FLAG")
+		(at 59.69 26.67 0)
+		(unit 1)
+		(exclude_from_sim no)
+		(in_bom yes)
+		(on_board yes)
+		(dnp no)
+		(fields_autoplaced yes)
+		(property "Reference" "#FLG01"
+			(at 59.69 24.765 0)
+			(effects
+				(font
+					(size 1.27 1.27)
+				)
+				(hide yes)
+			)
+		)
+		(property "Value" "PWR_FLAG"
+			(at 59.69 21.59 0)
+			(effects
+				(font
+					(size 1.27 1.27)
+				)
+			)
+		)
+		(property "Footprint" ""
+			(at 59.69 26.67 0)
+			(effects
+				(font
+					(size 1.27 1.27)
+				)
+				(hide yes)
+			)
+		)
+		(property "Datasheet" "~"
+			(at 59.69 26.67 0)
+			(effects
+				(font
+					(size 1.27 1.27)
+				)
+				(hide yes)
+			)
+		)
+		(property "Description" "Special symbol for telling ERC where power comes from"
+			(at 59.69 26.67 0)
+			(effects
+				(font
+					(size 1.27 1.27)
+				)
+				(hide yes)
+			)
+		)
+		(pin "1"
+		)
+		(instances
+			(project ""
+				(path "/e72bc999-a506-4a63-8c4b-c84561b55f6d/3bb3cd23-0a7e-4579-8d0d-52812beb7407"
+					(reference "#FLG01")
 					(unit 1)
 				)
@@
 		(on_board yes)
 		(dnp no)
-		(property "Reference" "#PWR035"
+		(property "Reference" "#PWR056"
 			(at 101.6 38.1 0)
 			(effects
@@
 			(project "sx1262xBoard"
 				(path "/e72bc999-a506-4a63-8c4b-c84561b55f6d/3bb3cd23-0a7e-4579-8d0d-52812beb7407"
-					(reference "#PWR035")
+					(reference "#PWR056")
 					(unit 1)
 				)
@@
 		(dnp no)
 		(fields_autoplaced yes)
-		(property "Reference" "#PWR037"
+		(property "Reference" "#PWR058"
 			(at 105.41 49.53 0)
 			(effects
@@
 			(project "sx1262xBoard"
 				(path "/e72bc999-a506-4a63-8c4b-c84561b55f6d/3bb3cd23-0a7e-4579-8d0d-52812beb7407"
-					(reference "#PWR037")
+					(reference "#PWR058")
 					(unit 1)
 				)
@@
 		(dnp no)
 		(fields_autoplaced yes)
-		(property "Reference" "#PWR033"
+		(property "Reference" "#PWR054"
 			(at 34.29 104.14 0)
 			(effects
@@
 			(project "sx1262xBoard"
 				(path "/e72bc999-a506-4a63-8c4b-c84561b55f6d/3bb3cd23-0a7e-4579-8d0d-52812beb7407"
-					(reference "#PWR033")
+					(reference "#PWR054")
 					(unit 1)
 				)
@@
 		(dnp no)
 		(fields_autoplaced yes)
-		(property "Reference" "R5"
+		(property "Reference" "R7"
 			(at 107.95 36.8299 0)
 			(effects
@@
 			(project "sx1262xBoard"
 				(path "/e72bc999-a506-4a63-8c4b-c84561b55f6d/3bb3cd23-0a7e-4579-8d0d-52812beb7407"
-					(reference "R5")
+					(reference "R7")
 					(unit 1)
 				)
@@
 		(dnp no)
 		(fields_autoplaced yes)
-		(property "Reference" "J2"
+		(property "Reference" "J3"
 			(at 38.1 19.05 0)
 			(effects
@@
 			(project "sx1262xBoard"
 				(path "/e72bc999-a506-4a63-8c4b-c84561b55f6d/3bb3cd23-0a7e-4579-8d0d-52812beb7407"
-					(reference "J2")
+					(reference "J3")
 					(unit 1)
 				)
@@
 		(dnp no)
 		(fields_autoplaced yes)
-		(property "Reference" "R6"
+		(property "Reference" "R8"
 			(at 119.38 34.2899 0)
 			(effects
@@
 			(project "sx1262xBoard"
 				(path "/e72bc999-a506-4a63-8c4b-c84561b55f6d/3bb3cd23-0a7e-4579-8d0d-52812beb7407"
-					(reference "R6")
+					(reference "R8")
 					(unit 1)
 				)
