File: sx1262x.kicad_sch (KiCad schematic)
At the start: 37 parts

Commit message: finalizing schematic
Parts:
- gave numbers to parts that had none: 37
Connections:
- net sxMOSI: no longer U1.16 (MISO)
- net ANTSwitch renamed DIO2
- new net sxMISO: U1.16 (MISO)
