File: sx1262xBoard.kicad_sch (KiCad schematic)
At the start: 0 parts

Commit message: finalizing schematic
Other:
- added sheet CAN (CAN.kicad_sch)
- added sheet Power (Power.kicad_sch)
- sheet FlashSD ports: added SDCLK, SDMISO, SDMOSI; removed none
- sheet MCU ports: added CAN_RX_2, CAN_TX_2, D+, D-, SPI2_MISO, SPI2_MOSI, SPI2_SCK, SPI_MISO, SPI_MOSI, SPI_SCK, SxBusy, SxDIO1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; removed none
- sheet USB_C ports: added D+, D-, VBUS; removed none
- sheet sx1262x ports: added sxBusy, sxDIO1, sxMISO, sxMOSI, sxNSS, sxReset, sxSCK; removed none
